File: NV08C_GPS_shield.sch (EAGLE design)
At the start: 65 parts, among them IC1 MCP1702-3.3, IC2 74LVC1T45SOT23-HAND, IC3 74LVC1T45SOT23-HAND, IC4 74LVC1T45SOT23-HAND, IC5 74LVC1T45SOT23-HAND, IC6 74LVC1T45SOT23-HAND, IC7 74LVC1T45SOT23-HAND, X1 MEGA2560, X2 CONN-SMATHD-SMD-EDGE, X4 UFL

Commit message: Minor layout changes.
Parts:
- X2: value CONN-SMATHD-SMD-EDGE -> CONN-SMATHD; device SteveMarple:CONN-SMATHD-SMD-EDGE -> SteveMarple:CONN-SMATHD
Changed lines of the file:
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@@
 <grid distance="0.1" unitdist="inch" unit="inch" style="lines" multiple="1" display="no" altdistance="0.01" altunitdist="inch" altunit="inch"/>
 <layers>
-<layer number="1" name="Top" color="4" fill="1" visible="no" active="no"/>
-<layer number="2" name="Route2" color="1" fill="3" visible="no" active="no"/>
-<layer number="3" name="Route3" color="4" fill="3" visible="no" active="no"/>
-<layer number="14" name="Route14" color="1" fill="6" visible="no" active="no"/>
-<layer number="15" name="Route15" color="4" fill="6" visible="no" active="no"/>
-<layer number="16" name="Bottom" color="1" fill="1" visible="no" active="no"/>
-<layer number="17" name="Pads" color="2" fill="1" visible="no" active="no"/>
-<layer number="18" name="Vias" color="2" fill="1" visible="no" active="no"/>
-<layer number="19" name="Unrouted" color="6" fill="1" visible="no" active="no"/>
-<layer number="20" name="Dimension" color="15" fill="1" visible="no" active="no"/>
-<layer number="21" name="tPlace" color="7" fill="1" visible="no" active="no"/>
-<layer number="22" name="bPlace" color="7" fill="1" visible="no" active="no"/>
-<layer number="23" name="tOrigins" color="15" fill="1" visible="no" active="no"/>
-<layer number="24" name="bOrigins" color="15" fill="1" visible="no" active="no"/>
-<layer number="25" name="tNames" color="7" fill="1" visible="no" active="no"/>
-<layer number="26" name="bNames" color="7" fill="1" visible="no" active="no"/>
-<layer number="27" name="tValues" color="7" fill="1" visible="no" active="no"/>
-<layer number="28" name="bValues" color="7" fill="1" visible="no" active="no"/>
+<layer number="1" name="Top" color="4" fill="1" visible="yes" active="no"/>
+<layer number="2" name="Route2" color="1" fill="3" visible="yes" active="no"/>
+<layer number="3" name="Route3" color="4" fill="3" visible="yes" active="no"/>
+<layer number="14" name="Route14" color="1" fill="6" visible="yes" active="no"/>
+<layer number="15" name="Route15" color="4" fill="6" visible="yes" active="no"/>
+<layer number="16" name="Bottom" color="1" fill="1" visible="yes" active="no"/>
+<layer number="17" name="Pads" color="2" fill="1" visible="yes" active="no"/>
+<layer number="18" name="Vias" color="2" fill="1" visible="yes" active="no"/>
+<layer number="19" name="Unrouted" color="6" fill="1" visible="yes" active="no"/>
+<layer number="20" name="Dimension" color="15" fill="1" visible="yes" active="no"/>
+<layer number="21" name="tPlace" color="7" fill="1" visible="yes" active="no"/>
+<layer number="22" name="bPlace" color="7" fill="1" visible="yes" active="no"/>
+<layer number="23" name="tOrigins" color="15" fill="1" visible="yes" active="no"/>
+<layer number="24" name="bOrigins" color="15" fill="1" visible="yes" active="no"/>
+<layer number="25" name="tNames" color="7" fill="1" visible="yes" active="no"/>
+<layer number="26" name="bNames" color="7" fill="1" visible="yes" active="no"/>
+<layer number="27" name="tValues" color="7" fill="1" visible="yes" active="no"/>
+<layer number="28" name="bValues" color="7" fill="1" visible="yes" active="no"/>
 <layer number="29" name="tStop" color="7" fill="3" visible="no" active="no"/>
 <layer number="30" name="bStop" color="7" fill="6" visible="no" active="no"/>
@@
 <layer number="35" name="tGlue" color="7" fill="4" visible="no" active="no"/>
 <layer number="36" name="bGlue" color="7" fill="5" visible="no" active="no"/>
-<layer number="37" name="tTest" color="7" fill="1" visible="no" active="no"/>
-<layer number="38" name="bTest" color="7" fill="1" visible="no" active="no"/>
+<layer number="37" name="tTest" color="7" fill="1" visible="yes" active="no"/>
+<layer number="38" name="bTest" color="7" fill="1" visible="yes" active="no"/>
 <layer number="39" name="tKeepout" color="4" fill="11" visible="no" active="no"/>
 <layer number="40" name="bKeepout" color="1" fill="11" visible="no" active="no"/>
@@
 <layer number="44" name="Drills" color="7" fill="1" visible="no" active="no"/>
 <layer number="45" name="Holes" color="7" fill="1" visible="no" active="no"/>
-<layer number="46" name="Milling" color="3" fill="1" visible="no" active="no"/>
-<layer number="47" name="Measures" color="7" fill="1" visible="no" active="no"/>
-<layer number="48" name="Document" color="7" fill="1" visible="no" active="no"/>
-<layer number="49" name="Reference" color="7" fill="1" visible="no" active="no"/>
-<layer number="50" name="dxf" color="7" fill="1" visible="no" active="no"/>
-<layer number="51" name="tDocu" color="7" fill="1" visible="no" active="no"/>
-<layer number="52" name="bDocu" color="7" fill="1" visible="no" active="no"/>
-<layer number="53" name="tGND_GNDA" color="7" fill="9" visible="no" active="no"/>
-<layer number="54" name="bGND_GNDA" color="1" fill="9" visible="no" active="no"/>
-<layer number="56" name="wert" color="7" fill="1" visible="no" active="no"/>
-<layer number="57" name="tCAD" color="7" fill="1" visible="no" active="no"/>
+<layer number="46" name="Milling" color="3" fill="1" visible="yes" active="no"/>
+<layer number="47" name="Measures" color="7" fill="1" visible="yes" active="no"/>
+<layer number="48" name="Document" color="7" fill="1" visible="yes" active="no"/>
+<layer number="49" name="Reference" color="7" fill="1" visible="yes" active="no"/>
+<layer number="50" name="dxf" color="7" fill="1" visible="yes" active="no"/>
+<layer number="51" name="tDocu" color="7" fill="1" visible="yes" active="no"/>
+<layer number="52" name="bDocu" color="7" fill="1" visible="yes" active="no"/>
+<layer number="53" name="tGND_GNDA" color="7" fill="9" visible="yes" active="no"/>
+<layer number="54" name="bGND_GNDA" color="1" fill="9" visible="yes" active="no"/>
+<layer number="56" name="wert" color="7" fill="1" visible="yes" active="no"/>
+<layer number="57" name="tCAD" color="7" fill="1" visible="yes" active="no"/>
 <layer number="91" name="Nets" color="2" fill="1" visible="yes" active="yes"/>
 <layer number="92" name="Busses" color="1" fill="1" visible="yes" active="yes"/>
@@
 <part name="U$15" library="SteveMarple" deviceset="PAD" device=""/>
 <part name="GND7" library="supply1" deviceset="GND" device=""/>
-<part name="X2" library="SteveMarple" deviceset="CONN-SMA" device="THD-SMD-EDGE"/>
+<part name="X2" library="SteveMarple" deviceset="CONN-SMA" device="THD" value="CONN-SMATHD"/>
 <part name="JP6" library="SparkFun" deviceset="JUMPER-3" device="PTH" value="V ANT"/>
 <part name="+3V2" library="supply1" deviceset="+3V3" device=""/>

Commit message: Fixing existing comments and adding new ones.
Parts:
- C10, C11: value 100n -> 1u
- C12, C9: value 100n -> 22p; device SteveMarple:C-EU1206-HAND -> SteveMarple:C-EU0805-HAND
- C13: value 1u -> 22p; device SteveMarple:C-EU1206-HAND -> SteveMarple:C-EU0805-HAND
- C3, C5, C6: value 1u -> 100n
- C4: value 22p -> 100n; device SteveMarple:C-EU0805-HAND -> SteveMarple:C-EU1206-HAND
- C7, C8: value 22p -> 1u; device SteveMarple:C-EU0805-HAND -> SteveMarple:C-EU1206-HAND
- U$10: value ? -> PAD
- U$11: value PAD -> CALUNIUM-SHIELD-V3V3-NO-HOLES-NO-TEXT; device SteveMarple:PAD -> SteveMarple:CALUNIUM-SHIELD-V3V3-NO-HOLES-NO-TEXT
- U$20: value PAD -> ?
- U$5: value CALUNIUM-SHIELD-V3V3-NO-HOLES-NO-TEXT -> PAD; device SteveMarple:CALUNIUM-SHIELD-V3V3-NO-HOLES-NO-TEXT -> SteveMarple:PAD
- renumbered X4 to X3
Connections:
- net !RESET: now also U$11.!RESET@0, U$11.!RESET@1; no longer U$5.!RESET@0, U$5.!RESET@1
- net +3V3: now also C10.1, C8.1, C9.1; no longer C12.1, C13.1, C4.1
- net +5V: now also C7.1, U$1.1, U$11.5V; no longer C2.1, U$17.1, U$5.5V
- net 11: now also U$11.11(MOSI); no longer U$5.11(MOSI)
- net 12: now also U$11.12(MISO); no longer U$5.12(MISO)
- net 13: now also U$11.13(SCK); no longer U$5.13(SCK)
- net 3V3_SHIELD: now also U$11.3.3V, U$2.1; no longer U$16.1, U$5.3.3V
- net 6: now also U$11.6; no longer U$5.6
- net 7: now also U$11.7; no longer U$5.7
- net A0: now also U$11.A0; no longer U$5.A0
- net GND: now also C7.2, U$11.GND, U$12.1, U$17.1; no longer C12.2, U$18.1, U$25.1, U$5.GND
- net GPIO0: now also U$18.1; no longer U$8.1
- net GPIO1: now also U$19.1; no longer U$9.1
- net GPIO2: now also U$20.1; no longer U$10.1
- net GPIO3: now also U$21.1; no longer U$11.1
- net GPIO4: now also U$22.1; no longer U$12.1
- net GPIO5: now also U$23.1; no longer U$13.1
- net GPIO6: now also U$24.1; no longer U$14.1
- net GPIO7: now also U$25.1; no longer U$15.1
- net IOREF: now also C3.1, C4.1, U$11.IOREF, U$13.1; no longer C10.1, C9.1, U$5.IOREF, U$6.1
- net ISP_VCC: now also U$11.ISP_VCC; no longer U$5.ISP_VCC
- net MEGA_28: now also U$14.1; no longer U$24.1
- net MEGA_30: now also U$15.1; no longer U$23.1
- net MISO: now also U$11.ISP_MISO; no longer U$5.ISP_MISO
- net MOSI: now also U$11.ISP_MOSI; no longer U$5.ISP_MOSI
- net N$1: now also C2.1; no longer C3.1
- net N$10: now also U$11.16, U$3.1; no longer U$22.1, U$5.16
- net N$2: now also U$11.19, U$6.1; no longer U$19.1, U$5.19
- net N$4: now also C12.2; no longer C7.2
- net N$6: now also U$11.18, U$5.1; no longer U$20.1, U$5.18
- net N$7: now also C12.1; no longer C7.1
- net N$9: now also U$11.17, U$4.1; no longer U$21.1, U$5.17
- net RX0: now also U$11.0(RX0), U$7.1; no longer U$1.1, U$5.0(RX0)
- net RX1: now also U$11.2(RX1)@1, U$9.1; no longer U$3.1, U$5.2(RX1)@1
- net SCK: now also U$11.ISP_SCK; no longer U$5.ISP_SCK
- net SLEEP_FLAG: now also U$16.1; no longer U$7.1
- net TX0: now also U$11.1(TX0), U$8.1; no longer U$2.1, U$5.1(TX0)
- net TX1: now also U$10.1, U$11.3(TX1)@1; no longer U$4.1, U$5.3(TX1)@1
- net V_ANT: now also C13.1; no longer C8.1
Other:
- note added: "Fit shunts to adjust default configuration (see datasheet). Makes use of internal pull-ups and pull-downs."
- note added: "Jumper block means a stacking ISP header is not needed. Fit shunts for Calunium and standare Arduino, omit for use with Arduino Mega2560."
- note added: "RF supply decoupling, position close to VIN_A pin."
- note added: "Use TO-92 package for better power dissapation."
- note removed: "Add other INT pin for Mega"
- note removed: "Position close to VIN_A pin."
- note removed: "Use TO-95 package for better power dissapation."
- moved on the sheet: C1, C10, C11, C12, C13, C2, C3, C4, C5, C6, C7, C8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
